File: PCB/Hyper_Wheel-base/Hyper_Wheel-base.kicad_pcb (KiCad board)
At the start: 4 copper layers, 81.9 x 68 mm, 77 parts, among them J1-1 Conn_01x06_Socket, J2 LIPO, J2-1 Conn_01x04_Socket, J3 USB4215-03-A, SW1 SW_Push, SW2 SW_Push, U1 CSD85301Q2, U10 TPS22916CNYFPR, U11 TPD2EUSB30ADRTR, U13 AS5600L-ASOM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

Commit message: Added test pads,
Parts:
- added P1: TestPad, TestPoint:TestPoint_Pad_D1.0mm, F.Cu at (213.5, 68.2)
- added P10: TestPad, TestPoint:TestPoint_Pad_D1.0mm, F.Cu at (218.2, 68.2)
- added P11: TestPad, TestPoint:TestPoint_Pad_D1.0mm, F.Cu at (219.2, 71.8)
- added P12: TestPad, TestPoint:TestPoint_Pad_D1.0mm, F.Cu at (216.8, 71.8)
- added P15: TestPad, TestPoint:TestPoint_Pad_D1.0mm, F.Cu at (179.2, 54.2)
- added P16: TestPad, TestPoint:TestPoint_Pad_D1.0mm, F.Cu at (212.2, 76.5)
- added P17: TestPad, TestPoint:TestPoint_Pad_D1.0mm, F.Cu at (178.0, 68.5)
- added P18: TestPad, TestPoint:TestPoint_Pad_D1.0mm, F.Cu at (180.2, 68.5)
- added P19: TestPad, TestPoint:TestPoint_Pad_D1.0mm, F.Cu at (214.2, 71.8)
- added P2: TestPad, TestPoint:TestPoint_Pad_D1.0mm, F.Cu at (210.8, 68.2)
- added P21: TestPad, TestPoint:TestPoint_Pad_D1.0mm, F.Cu at (240.5, 70.2)
- added P22: TestPad, TestPoint:TestPoint_Pad_D1.0mm, F.Cu at (237.5, 70.2)
- added P23: TestPad, TestPoint:TestPoint_Pad_D1.0mm, F.Cu at (220.2, 76.5)
- added P24: TestPad, TestPoint:TestPoint_Pad_D1.0mm, F.Cu at (216.5, 76.5)
- added P3: TestPad, TestPoint:TestPoint_Pad_D1.0mm, F.Cu at (215.8, 53.5)
- added P4: TestPad, TestPoint:TestPoint_Pad_D1.0mm, F.Cu at (218.8, 53.5)
- added P5: TestPad, TestPoint:TestPoint_Pad_D1.0mm, F.Cu at (213.2, 57.8)
- added P6: TestPad, TestPoint:TestPoint_Pad_D1.0mm, F.Cu at (216.0, 68.2)
- added P7: TestPad, TestPoint:TestPoint_Pad_D1.0mm, F.Cu at (212.8, 53.5)
- added P8: TestPad, TestPoint:TestPoint_Pad_D1.0mm, F.Cu at (218.5, 61.0)
- added P9: TestPad, TestPoint:TestPoint_Pad_D1.0mm, F.Cu at (215.5, 59.5)
- moved SW2 3.25 mm to (179.7, 63.1)
- moved SW1 3.25 mm to (179.7, 63.1)
- moved J2 2.15 mm to (179.5, 72.8)
Connections:
- U2 pad AA24: unconnected-(U2C-SWDCLK-PadAA24) -> Net-(P21-Pin_1)
- U2 pad AC17: unconnected-(U2A-P0.21-PadAC17) -> /Spare1
- U2 pad AC19: unconnected-(U2A-P0.23-PadAC19) -> /Spare2
- U2 pad AC24: unconnected-(U2C-SWDIO-PadAC24) -> Net-(P22-Pin_1)
- U2 pad D2: Net-(U2B-P0.00/XL1) -> /Net-(U2B-P0.00/XL1)
- U2 pad F2: Net-(U2B-P0.01/XL2) -> /Net-(U2B-P0.01/XL2)
- U2 pad H23: Net-(U2B-ANT) -> /Net-(U2B-ANT)
Routing:
- net /Spare2: track 0.00 -> 26.2 mm, vias 0 -> 2
- net /Spare1: track 0.00 -> 21.1 mm, vias 0 -> 2
- net Net-(P21-Pin_1): track 0.00 -> 9.33 mm
- net /Power Handling/Cell-: track 22.6 -> 29.3 mm
- net Net-(P22-Pin_1): track 0.00 -> 6.23 mm
- net /Power Handling/Cell+: track 36.7 -> 41.7 mm
- net /I2C_1_SCL: track 43.2 -> 47.8 mm
- net /I2C_1_SDA: track 42.5 -> 46.0 mm
- net /Switch: track 62.7 -> 65.9 mm
- net Net-(U2A-P0.18/~{RESET}): track 60.7 -> 64.0 mm
- net /I2C_2_SDA: track 61.5 -> 64.5 mm, vias 3 -> 4
- net /Load1 CTRL: track 10.7 -> 13.5 mm, vias 0 -> 2
- net /Load2 CTRL: track 13.2 -> 15.8 mm, vias 0 -> 2
- net /I2C_2_SCL: track 61.3 -> 63.4 mm
- net ChargerOUT: track 27.2 -> 28.9 mm
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