File: PCB/Hyper_Wheel-base/Hyper_Wheel-base.kicad_pcb (KiCad board)
At the start: 4 copper layers, 95 x 68 mm, 94 parts, among them J1-1 Conn_01x06_Socket, J2 LIPO, J2-1 Conn_01x04_Socket, J3 USB4215-03-A, P1 TestPad, P10 TestPad, P11 TestPad, P12 TestPad, P15 TestPad, P16 TestPad, P17 TestPad, P18 TestPad, P19 TestPad, P2 TestPad, P21 TestPad, P22 TestPad, P23 TestPad, P24 TestPad, P3 TestPad, P4 TestPad, P5 TestPad, P6 TestPad, P7 TestPad, P8 TestPad, P9 TestPad, SW1 SW_Push, SW2 SW_Push, U1 CSD85301Q2, U10 TPS22916CNYFPR, U11 TPD2EUSB30ADRTR, U17 2450AT07A0100T, U2 NRF52840-QIAA-R7, U4 TPS22916CNYFPR, U6 BQ29700DSER, U7 BQ24074RGTR, U9 CSD85301Q2, Y1 32MHz

Commit message: fabrication submit for XIAO and encoder wheels
Parts:
- added JP1: Jumper_2_Open, Jumper:SolderJumper-2_P1.3mm_Open_Pad1.0x1.5mm, B.Cu at (184.2, 60.4)
- added JP2: Jumper_2_Open, Jumper:SolderJumper-2_P1.3mm_Open_Pad1.0x1.5mm, B.Cu at (184.2, 56.9)
Routing:
- net /Load2 V: track 43.1 -> 16.3 mm
- net /I2C_2_SDA: track 64.5 -> 84.0 mm
- net /I2C_2_SCL: track 63.4 -> 77.7 mm
- net /I2C_1_SCL: track 47.8 -> 56.7 mm
- net /I2C_1_SDA: track 46.0 -> 53.7 mm

Commit message: Final cleanup
Parts:
- renumbered P11 to 3.3V, P9 to CM, P6 to CT1, P8 to CT2, P19 to Cell+, P16 to G, P10 to Hall, P5 to Load1, P7 to Load2, R_I2c_2 to RD1, R_I2c_3 to RD2, R_I2c_1 to RS1, R_I2c_4 to RS2, P2 to SCL1, P3 to SCL2, P1 to SDA1, P4 to SDA2, P23 to Sp1, P24 to Sp2, P12 to VB
Routing:
- net ChargerOUT: track 28.9 -> 26.8 mm
- net /D+: track 22.6 -> 20.5 mm
- net Net-(U1A-G1): track 5.02 -> 6.52 mm, vias 0 -> 2
- net /USB Vbus: track 68.5 -> 69.5 mm
- net /I2C_2_SCL: track 77.7 -> 78.2 mm
- net /I2C_2_SDA: track 84.0 -> 83.5 mm
Other:
- outline, holes or cut-outs redrawn

Commit message: added Revision mark
Parts:
- added G***: LOGO, Hyper_Wheel:Goat, B.Cu at (235.4, 62.0)
