File: PCB/Hyper_Wheel-base/Hyper_Wheel-base.kicad_pcb (KiCad board)
At the start: 4 copper layers, 95 x 68 mm, 105 parts, among them J1-1 Conn_01x06_Socket, J2 LIPO, J2-1 Conn_01x04_Socket, J3 USB4215-03-A, P15 TestPad, P17 TestPad, P18 TestPad, P21 TestPad, P22 TestPad, SW1 SW_Push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

Commit message: Rev B Xiao.  migrated changes to main
Parts:
- added JP3: Jumper_3_Bridged12, Jumper:SolderJumper-3_P1.3mm_Bridged12_Pad1.0x1.5mm, B.Cu at (215.0, 49.0)
- added JP4: Jumper_3_Bridged12, Jumper:SolderJumper-3_P1.3mm_Bridged12_Pad1.0x1.5mm, B.Cu at (215.0, 51.5)
- CH1, CH2, CH3, CH4, CH5, CH6, CH7, CH8: footprint Hyper_Wheel:SW_KS33_HS_KS-2P02B01-02_HS_1u -> Hyper_Wheel:SW_KS33_1u
- moved CH1 1.00 mm to (186.0, 89.4), turned to 180 degrees
- moved CH2 1.00 mm to (206.0, 89.4), turned to 180 degrees
- moved CH3 1.00 mm to (226.0, 89.4), turned to 180 degrees
- moved CH4 1.00 mm to (246.0, 89.4), turned to 180 degrees
- moved CH5 1.00 mm to (186.0, 40.4)
- moved CH6 1.00 mm to (206.0, 40.4)
- moved CH7 1.00 mm to (226.0, 40.4)
- moved CH8 1.00 mm to (246.0, 40.3)
Connections:
- U15 pad 1: /Load2 V -> Net-(JP3-A)
- U15 pad 2: GND -> Net-(JP3-B)
- U16 pad 1: /Load2 V -> Net-(JP3-A)
- U16 pad 2: GND -> Net-(JP3-B)
Routing:
- net Net-(JP3-A): track 0.00 -> 49.6 mm, vias 0 -> 2
- net Net-(JP3-B): track 0.00 -> 47.5 mm, vias 0 -> 2
- net /Key7: track 16.7 -> 29.9 mm
- net /Key3: track 30.3 -> 20.9 mm
- net /Key5: track 50.6 -> 59.8 mm
- net /Key6: track 31.0 -> 40.2 mm
- net /Key2: track 49.0 -> 39.8 mm
- net /Key8: track 33.8 -> 25.4 mm
- net /Key4: track 41.3 -> 33.5 mm
- net /Key1: track 65.9 -> 59.6 mm
- net /Load2 V: track 7.98 -> 4.75 mm

Commit message: added .5mm pitch ribbon cable. install TBD
Parts:
- moved G*** 4.25 mm to (239.3, 63.5), turned to 180 degrees
Changed lines of the file:
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@@
 	(footprint "Hyper_Wheel:Goat"
 		(layer "B.Cu")
-		(at 235.402519 61.964966)
+		(at 239.347481 63.535035 180)
 		(property "Reference" "G***"
 			(at 0 0 0)
@@
 		(fp_poly
 			(pts
-				(xy -2.955192 4.530481) (xy -2.967404 4.51827) (xy -2.979615 4.530481) (xy -2.967404 4.542693)
+				(xy 1.440961 4.823558) (xy 1.42875 4.811347) (xy 1.416538 4.823558) (xy 1.42875 4.83577)
 			)
 			(stroke
@@
 		(fp_poly
 			(pts
-				(xy 1.440961 4.823558) (xy 1.42875 4.811347) (xy 1.416538 4.823558) (xy 1.42875 4.83577)
+				(xy -2.955192 4.530481) (xy -2.967404 4.51827) (xy -2.979615 4.530481) (xy -2.967404 4.542693)
 			)
 			(stroke
@@
 		)
 	)
+	(gr_text_box "VCCSW\nGND\nSDL\nSCA\nHall\nVCC"
+		(start 191.90625 55.533397)
+		(end 200.59375 72.466603)
+		(margins 1.0025 1.0025 1.0025 1.0025)
+		(layer "B.SilkS")
+		(effects
+			(font
+				(size 1.5 1.5)
+				(thickness 0.2)
+			)
+			(justify left top mirror)
+		)
+		(border yes)
+		(stroke
+			(width 0.1)
+			(type solid)
+		)
+		(knockout no)
+	)
 	(gr_text_box "Hyper-Wheel\nFull System\nRevA 1\n4/26"
-		(start 216.625 58.572084)
-		(end 228.875 66.927916)
+		(start 208.25 60.572084)
+		(end 225.125 72.278832)
 		(margins 1.0025 1.0025 1.0025 1.0025)
 		(layer "B.SilkS")
 		(effects
 			(font
-				(size 1 1)
-				(thickness 0.1)
+				(size 1.5 1.5)
+				(thickness 0.2)
 			)
 			(justify left top mirror)
