File: PCB/Hyper_Wheel-base/Hyper_Wheel-base.kicad_sch (KiCad schematic)
At the start: 31 parts, among them J3 USB4215-03-A, P1 TestPad, P10 TestPad, P11 TestPad, P12 TestPad, P15 TestPad, P16 TestPad, P2 TestPad, P23 TestPad, P24 TestPad, P3 TestPad, P4 TestPad, P5 TestPad, P6 TestPad, P7 TestPad, P8 TestPad, P9 TestPad, SW1 SW_Push, SW2 SW_Push, U11 TPD2EUSB30ADRTR, U17 2450AT07A0100T, U2 NRF52840-QIAA-R7

Commit message: XIAO based test board complete
Parts:
- D1, RCC1, RCC2, RUSB1, RUSB2, R_I2c_1, R_I2c_2, R_I2c_3, R_I2c_4: KiLib_Generator (none) -> SMD_2terminal_chip_molded
- P1: footprint TestPoint:TestPoint_Pad_D1.5mm -> TestPoint:TestPoint_Pad_D1.0mm; now left out of the parts list
- P10, P11, P12, P15, P16, P2, P23, P24, P3, P4, P5, P6, P7, P8, P9: footprint TestPoint:TestPoint_Pad_D2.0mm -> TestPoint:TestPoint_Pad_D1.0mm; now left out of the parts list
- U11: KiLib_Generator (none) -> package/gullwing

Commit message: fabrication submit for XIAO and encoder wheels
Parts:
- added JP1, JP2: Jumper_2_Open, Jumper:SolderJumper-2_P1.3mm_Open_Pad1.0x1.5mm, symbol Jumper:Jumper_2_Open
Connections:
- net I2C_1_SCL: now also JP2.2 (B)
- net I2C_1_SDA: now also JP1.2 (B)
- net I2C_2_SCL: now also JP2.1 (A)
- net I2C_2_SDA: now also JP1.1 (A)
Changed lines of the file:
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@@
 	(wire
 		(pts
+			(xy 66.04 48.26) (xy 73.66 48.26)
+		)
+		(stroke
+			(width 0)
+			(type default)
+		)
+	)
+	(wire
+		(pts
 			(xy 95.25 85.09) (xy 86.36 85.09)
 		)
@@
 	(wire
 		(pts
+			(xy 44.45 57.15) (xy 55.88 57.15)
+		)
+		(stroke
+			(width 0)
+			(type default)
+		)
+	)
+	(wire
+		(pts
 			(xy 147.32 163.83) (xy 147.32 176.53)
 		)
@@
 	(wire
 		(pts
+			(xy 43.18 48.26) (xy 55.88 48.26)
+		)
+		(stroke
+			(width 0)
+			(type default)
+		)
+	)
+	(wire
+		(pts
 			(xy 138.43 165.1) (xy 138.43 176.53)
 		)
@@
 		)
 	)
+	(wire
+		(pts
+			(xy 66.04 57.15) (xy 71.12 57.15)
+		)
+		(stroke
+			(width 0)
+			(type default)
+		)
+	)
 	(image
 		(at 252.73 134.62)
@@
 		)
 	)
+	(label "I2C_2_SCL"
+		(at 44.45 57.15 0)
+		(effects
+			(font
+				(size 1.27 1.27)
+			)
+			(justify left bottom)
+		)
+	)
 	(label "Load3 V"
 		(at 132.08 173.99 90)
@@
 		)
 	)
+	(label "I2C_1_SCL"
+		(at 71.12 57.15 0)
+		(effects
+			(font
+				(size 1.27 1.27)
+			)
+			(justify left bottom)
+		)
+	)
 	(label "Hall_1"
 		(at 113.03 166.37 0)
@@
 		)
 	)
+	(label "I2C_2_SDA"
+		(at 43.18 48.26 0)
+		(effects
+			(font
+				(size 1.27 1.27)
+			)
+			(justify left bottom)
+		)
+	)
 	(label "Key7"
 		(at 173.99 171.45 90)
@@
 		)
 	)
+	(label "I2C_1_SDA"
+		(at 73.66 48.26 0)
+		(effects
+			(font
+				(size 1.27 1.27)
+			)
+			(justify left bottom)
+		)
+	)
 	(label "Load1 V"
 		(at 17.78 170.18 90)
@@
 	)
 	(symbol
+		(lib_id "Jumper:Jumper_2_Open")
+		(at 60.96 48.26 0)
+		(unit 1)
+		(body_style 1)
+		(exclude_from_sim no)
+		(in_bom yes)
+		(on_board yes)
+		(in_pos_files yes)
+		(dnp no)
+		(fields_autoplaced yes)
+		(property "Reference" "JP1"
+			(at 60.96 41.91 0)
+			(show_name no)
+			(do_not_autoplace no)
+			(effects
+				(font
+					(size 1.27 1.27)
+				)
+			)
+		)
+		(property "Value" "Jumper_2_Open"
+			(at 60.96 44.45 0)
+			(show_name no)
+			(do_not_autoplace no)
+			(effects
+				(font
+					(size 1.27 1.27)
+				)
+			)
+		)
+		(property "Footprint" "Jumper:SolderJumper-2_P1.3mm_Open_Pad1.0x1.5mm"
+			(at 60.96 48.26 0)
+			(hide yes)
+			(show_name no)
+			(do_not_autoplace no)
+			(effects
+				(font
+					(size 1.27 1.27)
+				)
+			)
+		)
+		(property "Datasheet" ""
+			(at 60.96 48.26 0)
+			(hide yes)
+			(show_name no)
+			(do_not_autoplace no)
+			(effects
+				(font
+					(size 1.27 1.27)
+				)
+			)
+		)
+		(property "Description" "Jumper, 2-pole, open"
+			(at 60.96 48.26 0)
+			(hide yes)
+			(show_name no)
+			(do_not_autoplace no)
+			(effects
+				(font
+					(size 1.27 1.27)
+				)
+			)
+		)
+		(pin "2"
+		)
+		(pin "1"
+		)
+		(instances
+			(project "Hyper_Wheel-base"
+				(path "/3f05eeb1-03f9-49d1-8a58-0bc3d5427d25"
+					(reference "JP1")
+					(unit 1)
+				)
+			)
+		)
+	)
+	(symbol
 		(lib_id "Connector:Conn_01x01_Pin")
 		(at 139.7 20.32 0)
@@
 					(unit 1)
 				)
+			)
+		)
+	)
+	(symbol
+		(lib_id "Jumper:Jumper_2_Open")
+		(at 60.96 57.15 0)
+		(unit 1)
+		(body_style 1)
+		(exclude_from_sim no)
+		(in_bom yes)
+		(on_board yes)
+		(in_pos_files yes)
+		(dnp no)
+		(fields_autoplaced yes)
+		(property "Reference" "JP2"
+			(at 60.96 50.8 0)
+			(show_name no)
+			(do_not_autoplace no)
+			(effects
+				(font
+					(size 1.27 1.27)
+				)
+			)
+		)
+		(property "Value" "Jumper_2_Open"
+			(at 60.96 53.34 0)
+			(show_name no)
+			(do_not_autoplace no)
+			(effects
+				(font
+					(size 1.27 1.27)
+				)
+			)
+		)
+		(property "Footprint" "Jumper:SolderJumper-2_P1.3mm_Open_Pad1.0x1.5mm"
+			(at 60.96 57.15 0)
+			(hide yes)
+			(show_name no)
+			(do_not_autoplace no)
+			(effects
+				(font
+					(size 1.27 1.27)
+				)
+			)
+		)
+		(property "Datasheet" ""
+			(at 60.96 57.15 0)
+			(hide yes)
+			(show_name no)
+			(do_not_autoplace no)
+			(effects
+				(font
+					(size 1.27 1.27)
+				)
+			)
+		)
+		(property "Description" "Jumper, 2-pole, open"
+			(at 60.96 57.15 0)
+			(hide yes)
+			(show_name no)
+			(do_not_autoplace no)
+			(effects
+				(font
+					(size 1.27 1.27)
+				)
+			)
+		)
+		(pin "2"
+		)
+		(pin "1"
+		)
+		(instances
+			(project "Hyper_Wheel-base"
+				(path "/3f05eeb1-03f9-49d1-8a58-0bc3d5427d25"
+					(reference "JP2")
+					(unit 1)
+				)
