File: PCB/Hyper_Wheel-base/Hyper_Wheel-base.kicad_sch (KiCad schematic)
At the start: 33 parts, among them J3 USB4215-03-A, P1 TestPad, P10 TestPad, P11 TestPad, P12 TestPad, P15 TestPad, P16 TestPad, P2 TestPad, P23 TestPad, P24 TestPad, P3 TestPad, P4 TestPad, P5 TestPad, P6 TestPad, P7 TestPad, P8 TestPad, P9 TestPad, SW1 SW_Push, SW2 SW_Push, U11 TPD2EUSB30ADRTR, U17 2450AT07A0100T, U2 NRF52840-QIAA-R7

Commit message: Final cleanup
Parts:
- renumbered P11 to 3.3V, P9 to CM, P6 to CT1, P8 to CT2, P16 to G, P10 to Hall, P5 to Load1, P7 to Load2, R_I2c_2 to RD1, R_I2c_3 to RD2, R_I2c_1 to RS1, R_I2c_4 to RS2, P2 to SCL1, P3 to SCL2, P1 to SDA1, P4 to SDA2, P23 to Sp1, P24 to Sp2, P12 to VB
Changed lines of the file:
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@@
 		(dnp no)
 		(fields_autoplaced yes)
-		(property "Reference" "R_I2c_1"
+		(property "Reference" "RS1"
 			(at 185.42 100.33 90)
 			(show_name no)
@@
 			(project "Hyper_Wheel-base"
 				(path "/3f05eeb1-03f9-49d1-8a58-0bc3d5427d25"
-					(reference "R_I2c_1")
+					(reference "RS1")
 					(unit 1)
 				)
@@
 		(dnp no)
 		(fields_autoplaced yes)
-		(property "Reference" "R_I2c_2"
+		(property "Reference" "RD1"
 			(at 185.42 110.49 90)
 			(show_name no)
@@
 			(project "Hyper_Wheel-base"
 				(path "/3f05eeb1-03f9-49d1-8a58-0bc3d5427d25"
-					(reference "R_I2c_2")
+					(reference "RD1")
 					(unit 1)
 				)
@@
 		(dnp no)
 		(fields_autoplaced yes)
-		(property "Reference" "P3"
+		(property "Reference" "SCL2"
 			(at 66.675 25.4 0)
 			(show_name no)
@@
 			(project "Hyper_Wheel-base"
 				(path "/3f05eeb1-03f9-49d1-8a58-0bc3d5427d25"
-					(reference "P3")
+					(reference "SCL2")
 					(unit 1)
 				)
@@
 		(in_pos_files yes)
 		(dnp no)
-		(property "Reference" "P4"
+		(property "Reference" "SDA2"
 			(at 65.405 31.75 0)
 			(show_name no)
@@
 			(project "Hyper_Wheel-base"
 				(path "/3f05eeb1-03f9-49d1-8a58-0bc3d5427d25"
-					(reference "P4")
+					(reference "SDA2")
 					(unit 1)
 				)
@@
 		(dnp no)
 		(fields_autoplaced yes)
-		(property "Reference" "P6"
+		(property "Reference" "CT1"
 			(at 108.585 20.32 0)
 			(show_name no)
@@
 			(project "Hyper_Wheel-base"
 				(path "/3f05eeb1-03f9-49d1-8a58-0bc3d5427d25"
-					(reference "P6")
+					(reference "CT1")
 					(unit 1)
 				)
@@
 		(dnp no)
 		(fields_autoplaced yes)
-		(property "Reference" "P5"
+		(property "Reference" "Load1"
 			(at 108.585 15.24 0)
 			(show_name no)
@@
 			(project "Hyper_Wheel-base"
 				(path "/3f05eeb1-03f9-49d1-8a58-0bc3d5427d25"
-					(reference "P5")
+					(reference "Load1")
 					(unit 1)
 				)
@@
 		(dnp no)
 		(fields_autoplaced yes)
-		(property "Reference" "R_I2c_3"
+		(property "Reference" "RD2"
 			(at 185.42 120.65 90)
 			(show_name no)
@@
 			(project "Hyper_Wheel-base"
 				(path "/3f05eeb1-03f9-49d1-8a58-0bc3d5427d25"
-					(reference "R_I2c_3")
+					(reference "RD2")
 					(unit 1)
 				)
@@
 		(dnp no)
 		(fields_autoplaced yes)
-		(property "Reference" "P9"
+		(property "Reference" "CM"
 			(at 140.335 15.24 0)
 			(show_name no)
@@
 			(project "Hyper_Wheel-base"
 				(path "/3f05eeb1-03f9-49d1-8a58-0bc3d5427d25"
-					(reference "P9")
+					(reference "CM")
 					(unit 1)
 				)
@@
 		(dnp no)
 		(fields_autoplaced yes)
-		(property "Reference" "P8"
+		(property "Reference" "CT2"
 			(at 107.315 30.48 0)
 			(show_name no)
@@
 			(project "Hyper_Wheel-base"
 				(path "/3f05eeb1-03f9-49d1-8a58-0bc3d5427d25"
-					(reference "P8")
+					(reference "CT2")
 					(unit 1)
 				)
@@
 		(dnp no)
 		(fields_autoplaced yes)
-		(property "Reference" "P11"
+		(property "Reference" "3.3V"
 			(at 140.335 26.67 0)
 			(show_name no)
@@
 			(project "Hyper_Wheel-base"
 				(path "/3f05eeb1-03f9-49d1-8a58-0bc3d5427d25"
-					(reference "P11")
+					(reference "3.3V")
 					(unit 1)
 				)
@@
 		(dnp no)
 		(fields_autoplaced yes)
-		(property "Reference" "P7"
+		(property "Reference" "Load2"
 			(at 107.315 25.4 0)
 			(show_name no)
@@
 			(project "Hyper_Wheel-base"
 				(path "/3f05eeb1-03f9-49d1-8a58-0bc3d5427d25"
-					(reference "P7")
+					(reference "Load2")
 					(unit 1)
 				)
@@
 		(dnp no)
 		(fields_autoplaced yes)
-		(property "Reference" "R_I2c_4"
+		(property "Reference" "RS2"
 			(at 185.42 130.81 90)
 			(show_name no)
@@
 			(project "Hyper_Wheel-base"
 				(path "/3f05eeb1-03f9-49d1-8a58-0bc3d5427d25"
-					(reference "R_I2c_4")
+					(reference "RS2")
 					(unit 1)
 				)
@@
 		(dnp no)
 		(fields_autoplaced yes)
-		(property "Reference" "P16"
+		(property "Reference" "G"
 			(at 177.165 30.48 0)
 			(show_name no)
@@
 			(project "Hyper_Wheel-base"
 				(path "/3f05eeb1-03f9-49d1-8a58-0bc3d5427d25"
-					(reference "P16")
+					(reference "G")
 					(unit 1)
 				)
@@
 		(dnp no)
 		(fields_autoplaced yes)
-		(property "Reference" "P12"
+		(property "Reference" "VB"
 			(at 140.335 31.75 0)
 			(show_name no)
@@
 			(project "Hyper_Wheel-base"
 				(path "/3f05eeb1-03f9-49d1-8a58-0bc3d5427d25"
-					(reference "P12")
+					(reference "VB")
 					(unit 1)
 				)
@@
 		(in_pos_files yes)
 		(dnp no)
-		(property "Reference" "P23"
+		(property "Reference" "Sp1"
 			(at 193.802 16.764 0)
 			(show_name no)
@@
 			(project "Hyper_Wheel-base"
 				(path "/3f05eeb1-03f9-49d1-8a58-0bc3d5427d25"
-					(reference "P23")
+					(reference "Sp1")
 					(unit 1)
 				)
@@
 		(in_pos_files yes)
 		(dnp no)
-		(property "Reference" "P24"
+		(property "Reference" "Sp2"
 			(at 193.802 19.304 0)
 			(show_name no)
@@
 			(project "Hyper_Wheel-base"
 				(path "/3f05eeb1-03f9-49d1-8a58-0bc3d5427d25"
-					(reference "P24")
+					(reference "Sp2")
 					(unit 1)
 				)
@@
 		(dnp no)
 		(fields_autoplaced yes)
-		(property "Reference" "P1"
+		(property "Reference" "SDA1"
 			(at 67.945 13.97 0)
 			(show_name no)
@@
 			(project "Hyper_Wheel-base"
 				(path "/3f05eeb1-03f9-49d1-8a58-0bc3d5427d25"
-					(reference "P1")
+					(reference "SDA1")
 					(unit 1)
 				)
@@
 		(dnp no)
 		(fields_autoplaced yes)
-		(property "Reference" "P2"
+		(property "Reference" "SCL1"
 			(at 67.945 19.05 0)
 			(show_name no)
@@
 			(project "Hyper_Wheel-base"
 				(path "/3f05eeb1-03f9-49d1-8a58-0bc3d5427d25"
-					(reference "P2")
+					(reference "SCL1")
 					(unit 1)
 				)
@@
 		(dnp no)
 		(fields_autoplaced yes)
-		(property "Reference" "P10"
+		(property "Reference" "Hall"
 			(at 140.335 21.59 0)
 			(show_name no)
@@
 			(project "Hyper_Wheel-base"
 				(path "/3f05eeb1-03f9-49d1-8a58-0bc3d5427d25"
-					(reference "P10")
+					(reference "Hall")
 					(unit 1)
 				)
