File: PCB/Hyper_Wheel-base/Hyper_Wheel-base.kicad_sch (KiCad schematic)
At the start: 33 parts, among them J3 USB4215-03-A, P15 TestPad, SW1 SW_Push, SW2 SW_Push, U11 TPD2EUSB30ADRTR, U17 2450AT07A0100T, U2 NRF52840-QIAA-R7

Commit message: Switched Load switch update
Parts:
- renumbered 3.3V to 3.3V1, CM to CM1, G to G1, Hall to Hall1, VB to VB1
Changed lines of the file:
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@@
 		(dnp no)
 		(fields_autoplaced yes)
-		(property "Reference" "CM"
+		(property "Reference" "CM1"
 			(at 140.335 15.24 0)
 			(show_name no)
@@
 			(project "Hyper_Wheel-base"
 				(path "/3f05eeb1-03f9-49d1-8a58-0bc3d5427d25"
-					(reference "CM")
+					(reference "CM1")
 					(unit 1)
 				)
@@
 		(dnp no)
 		(fields_autoplaced yes)
-		(property "Reference" "3.3V"
+		(property "Reference" "3.3V1"
 			(at 140.335 26.67 0)
 			(show_name no)
@@
 			(project "Hyper_Wheel-base"
 				(path "/3f05eeb1-03f9-49d1-8a58-0bc3d5427d25"
-					(reference "3.3V")
+					(reference "3.3V1")
 					(unit 1)
 				)
@@
 		(dnp no)
 		(fields_autoplaced yes)
-		(property "Reference" "G"
+		(property "Reference" "G1"
 			(at 177.165 30.48 0)
 			(show_name no)
@@
 			(project "Hyper_Wheel-base"
 				(path "/3f05eeb1-03f9-49d1-8a58-0bc3d5427d25"
-					(reference "G")
+					(reference "G1")
 					(unit 1)
 				)
@@
 		(dnp no)
 		(fields_autoplaced yes)
-		(property "Reference" "VB"
+		(property "Reference" "VB1"
 			(at 140.335 31.75 0)
 			(show_name no)
@@
 			(project "Hyper_Wheel-base"
 				(path "/3f05eeb1-03f9-49d1-8a58-0bc3d5427d25"
-					(reference "VB")
+					(reference "VB1")
 					(unit 1)
 				)
@@
 		(dnp no)
 		(fields_autoplaced yes)
-		(property "Reference" "Hall"
+		(property "Reference" "Hall1"
 			(at 140.335 21.59 0)
 			(show_name no)
@@
 			(project "Hyper_Wheel-base"
 				(path "/3f05eeb1-03f9-49d1-8a58-0bc3d5427d25"
-					(reference "Hall")
-					(unit 1)
-				)
+					(reference "Hall1")
+					(unit 1)
+				)
