File: PCB/Encoder+Hall Breakout/Encoder+Hall Breakout.kicad_pcb (KiCad board)
At the start: 2 copper layers, 26.8 x 29.5 mm, 14 parts, among them J1-2 Conn_01x06_Pin, U1 AS5600L-ASOM, U2 DRV5032FCDBZR, U3 DRV5032FCDBZR

Commit message: fabrication submit for XIAO and encoder wheels
Parts:
- moved OUT1 1.31 mm to (143.2, 96.4)
- moved U1 0.17 mm to (132.3, 95.0)
Routing:
- net /OB-Hall: track 35.1 -> 36.6 mm
- net GND: track 5.04 -> 6.45 mm
- net Net-(U1-OUT): track 12.6 -> 11.3 mm
- net /OB-3.3v: track 43.2 -> 42.7 mm
Other:
- board size 26.8 x 29.5 mm -> 26.3 x 29.2 mm
