File: PCB/Hyper_Wheel_XIAO/Hyper_Wheel_XIAO.kicad_pcb (KiCad board)
At the start: 2 copper layers, 103.5 x 68 mm, 45 parts, among them J1-1 Conn_01x06_Socket, J2 LIPO, J2-1 Conn_01x04_Socket, P3 TestPad, P4 TestPad, SW2 SW_Push, U1 CSD85301Q2, U13 AS5600L-ASOM, U14 DRV5032FCDBZR, U2 Seeed Studio XIAO nRF52840, U3 AS5600L-ASOM, U6 BQ29700DSER, U8 DRV5032FCDBZR, U9 CSD85301Q2

Commit message: fabrication submit for XIAO and encoder wheels
Parts:
- JP4: moved to B.Cu
Routing:
- net /Cell-: vias 2 -> 3

Commit message: Rev B Xiao.  migrated changes to main
Parts:
- added JP1: Jumper_3_Bridged12, Jumper:SolderJumper-3_P1.3mm_Bridged12_Pad1.0x1.5mm_NumberLabels, B.Cu at (211.8, 56.8)
- added JP2: Jumper_3_Bridged12, Jumper:SolderJumper-3_P1.3mm_Bridged12_Pad1.0x1.5mm_NumberLabels, B.Cu at (209.0, 56.8)
- CH1, CH2, CH3, CH4, CH5, CH6, CH7, CH8: footprint Hyper_Wheel:SW_KS33_HS_KS-2P02B01-02_HS_1u -> Hyper_Wheel:SW_KS33_1u
- JP4: footprint Jumper:SolderJumper-2_P1.3mm_Open_Pad1.0x1.5mm -> Jumper:SolderJumper-2_P1.3mm_Bridged_Pad1.0x1.5mm
- RI1: renamed from R_I2c_1; footprint Resistor_SMD:R_0402_1005Metric -> Resistor_SMD:R_0603_1608Metric_Pad0.98x0.95mm_HandSolder
- RI2: renamed from R_I2c_2; footprint Resistor_SMD:R_0402_1005Metric -> Resistor_SMD:R_0603_1608Metric_Pad0.98x0.95mm_HandSolder
- Rdiv1, Rdiv2: footprint Resistor_SMD:R_0603_1608Metric -> Resistor_SMD:R_0603_1608Metric_Pad0.98x0.95mm_HandSolder
- moved CH1 1.00 mm to (186.0, 89.4), turned to 180 degrees
- moved CH2 1.00 mm to (206.0, 89.4), turned to 180 degrees
- moved CH3 1.00 mm to (226.0, 89.4), turned to 180 degrees
- moved CH4 1.00 mm to (246.0, 89.4), turned to 180 degrees
- moved CH5 1.00 mm to (186.0, 40.4)
- moved CH6 1.00 mm to (206.0, 40.4)
- moved CH7 1.00 mm to (226.0, 40.4)
- moved CH8 1.00 mm to (246.0, 40.3)
- renumbered P3 to SCL1, P4 to SDA1
Connections:
- U15 pad 1: 3.3V_Regulated -> Net-(JP1-A)
- U15 pad 2: GND -> Net-(JP1-B)
- U16 pad 1: 3.3V_Regulated -> Net-(JP1-A)
- U16 pad 2: GND -> Net-(JP1-B)
Routing:
- net Net-(JP1-B): track 0.00 -> 47.9 mm, vias 0 -> 4
- net Net-(JP1-A): track 0.00 -> 42.0 mm
- net /Key7: track 39.1 -> 47.9 mm
- net /Key6: track 57.2 -> 66.0 mm
- net /Key5: track 69.9 -> 78.7 mm
- net /Key4: track 25.3 -> 16.5 mm
- net /Key8: track 22.3 -> 30.3 mm
- net /Switch: track 100.3 -> 92.5 mm
- net /Key2: track 54.6 -> 52.6 mm
- net /Key3: track 36.9 -> 35.0 mm
- net GND: vias 0 -> 1

Commit message: RevB Xiao Updates. Fab
Parts:
- removed U13, U3: AS5600L-ASOM, Hyper_Wheel:AS5600L-ASOM_AMS
- removed U14, U8: DRV5032FCDBZR, Hyper_Wheel:DRV5032-DBZ0003A-IPC_A
- J1-1: footprint Connector_PinHeader_2.54mm:PinHeader_1x06_P2.54mm_Vertical -> Connector_JST:JST_EH_S6B-EH_1x06_P2.50mm_Horizontal; moved to B.Cu
- J2: footprint Connector_JST:JST_EH_B2B-EH-A_1x02_P2.50mm_Vertical -> Connector_JST:JST_EH_S2B-EH_1x02_P2.50mm_Horizontal; moved to B.Cu
- J2-1: footprint Connector_PinHeader_2.54mm:PinHeader_1x04_P2.54mm_Vertical -> Connector_JST:JST_EH_S4B-EH_1x04_P2.50mm_Horizontal; moved to B.Cu
- moved G*** 35.3 mm to (238.6, 68.5)
- moved J2-1 8.61 mm to (190.8, 66.0), turned to 90 degrees
- moved J2 4.25 mm to (179.5, 77.0)
- moved C- 4.03 mm to (176.8, 70.5)
- moved C+ 2.14 mm to (178.8, 70.5)
- moved J1-1 1.17 mm to (186.8, 58.5), turned to -90 degrees
- renumbered 3.3V1 to 3.3V, C+1 to C+, C-1 to C-, Cell1 to Cell, Cell+1 to Cell+, Cell-1 to Cell-, GND2 to GND, GND1 to GND, Hall1 to Hall, Hall2 to Hall, SCL1 to SCL, SDA1 to SDA, Switch1 to Switch
Routing:
- net /I2C_1_SDA: track 88.7 -> 91.6 mm, vias 2 -> 3
- net /Key5: track 78.7 -> 79.8 mm
- net ChargerOUT: track 114.2 -> 115.2 mm
- net /Power Handling/Cell-: track 38.3 -> 37.4 mm
- net /I2C_1_SCL: track 87.3 -> 88.1 mm
- net /Switch: track 92.5 -> 93.0 mm
- net Net-(U1A-G1): track 7.12 -> 7.69 mm
- net /Hall_1: track 65.5 -> 66.0 mm
Other:
- board text added: "C+ C-"
- board text added: "GND"
- board text added: "H1"
- board text added: "SDA SCL GND VCC"
- board text added: "VCC"
- board text added: "VCC SCL SDA Hall VCC"
