File: PCB/Hyper_Wheel_XIAO/Peripherals.kicad_sch (KiCad schematic)
At the start: 18 parts, among them J1-1 Conn_01x06_Socket, J1-2 Conn_01x06_Pin, J2-1 Conn_01x04_Socket, U13 AS5600L-ASOM, U14 DRV5032FCDBZR, U3 AS5600L-ASOM, U8 DRV5032FCDBZR

Commit message: Rev B Xiao.  migrated changes to main
Parts:
- added JP1, JP2: Jumper_3_Bridged12, Jumper:SolderJumper-3_P1.3mm_Bridged12_Pad1.0x1.5mm_NumberLabels, symbol Jumper:Jumper_3_Bridged12
Connections:
- net GND: now also JP1.2 (C); no longer U15.2 (GND), U16.2 (GND)
- net Load2_Vin: now also JP2.2 (C); no longer U15.1 (VCC), U16.1 (VCC)
- new net: JP1.1 (A), JP2.3 (B), U15.1 (GND), U16.1 (GND)
- new net: JP1.3 (B), JP2.1 (A), U15.2 (VCC), U16.2 (VCC)
Other:
- moved on the sheet: U15, U16

Commit message: RevB Xiao Updates. Fab
Parts:
- CH1, CH2, CH3, CH4, CH5, CH6, CH7, CH8: footprint Hyper_Wheel:SW_KS33_HS_KS-2P02B01-02_HS_1u -> Hyper_Wheel:SW_KS33_1u
- J1-1: footprint Connector_PinHeader_2.54mm:PinHeader_1x06_P2.54mm_Vertical -> Connector_JST:JST_EH_S6B-EH_1x06_P2.50mm_Horizontal
- J2-1: footprint Connector_PinHeader_2.54mm:PinHeader_1x04_P2.54mm_Vertical -> Connector_JST:JST_EH_S4B-EH_1x04_P2.50mm_Horizontal
Changed lines of the file:
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@@
+	(wire
+		(pts
+			(xy 106.68 153.67) (xy 106.68 156.21)
+		)
+		(stroke
+			(width 0)
+			(type default)
+		)
+	)
 	(wire
 		(pts
@@
 	(wire
 		(pts
+			(xy 106.68 161.29) (xy 119.38 161.29)
+		)
+		(stroke
+			(width 0)
+			(type default)
+		)
+	)
+	(wire
+		(pts
 			(xy 81.28 160.02) (xy 81.28 158.75)
 		)
@@
 	(wire
 		(pts
-			(xy 106.68 161.29) (xy 119.38 161.29)
-		)
-		(stroke
-			(width 0)
-			(type default)
-		)
-	)
-	(wire
-		(pts
 			(xy 246.38 166.37) (xy 246.38 162.56)
 		)
@@
 	(wire
 		(pts
+			(xy 247.65 140.97) (xy 247.65 139.7)
+		)
+		(stroke
+			(width 0)
+			(type default)
+		)
+	)
+	(wire
+		(pts
+			(xy 78.74 162.56) (xy 77.47 162.56)
+		)
+		(stroke
+			(width 0)
+			(type default)
+		)
+	)
+	(wire
+		(pts
+			(xy 118.11 57.15) (xy 129.54 57.15)
+		)
+		(stroke
+			(width 0)
+			(type default)
+		)
+	)
+	(wire
+		(pts
+			(xy 215.9 140.97) (xy 234.95 140.97)
+		)
+		(stroke
+			(width 0)
+			(type default)
+		)
+	)
+	(wire
+		(pts
+			(xy 143.51 59.69) (xy 154.94 59.69)
+		)
+		(stroke
+			(width 0)
+			(type default)
+		)
+	)
+	(wire
+		(pts
+			(xy 143.51 62.23) (xy 173.99 62.23)
+		)
+		(stroke
+			(width 0)
+			(type default)
+		)
+	)
+	(wire
+		(pts
+			(xy 218.44 54.61) (xy 232.41 54.61)
+		)
+		(stroke
+			(width 0)
+			(type default)
+		)
+	)
+	(wire
+		(pts
 			(xy 106.68 158.75) (xy 114.3 158.75)
 		)
@@
 	(wire
 		(pts
-			(xy 247.65 140.97) (xy 247.65 139.7)
-		)
-		(stroke
-			(width 0)
-			(type default)
-		)
-	)
-	(wire
-		(pts
-			(xy 78.74 162.56) (xy 77.47 162.56)
-		)
-		(stroke
-			(width 0)
-			(type default)
-		)
-	)
-	(wire
-		(pts
-			(xy 118.11 57.15) (xy 129.54 57.15)
-		)
-		(stroke
-			(width 0)
-			(type default)
-		)
-	)
-	(wire
-		(pts
-			(xy 215.9 140.97) (xy 234.95 140.97)
-		)
-		(stroke
-			(width 0)
-			(type default)
-		)
-	)
-	(wire
-		(pts
-			(xy 143.51 59.69) (xy 154.94 59.69)
-		)
-		(stroke
-			(width 0)
-			(type default)
-		)
-	)
-	(wire
-		(pts
-			(xy 143.51 62.23) (xy 173.99 62.23)
-		)
-		(stroke
-			(width 0)
-			(type default)
-		)
-	)
-	(wire
-		(pts
-			(xy 218.44 54.61) (xy 232.41 54.61)
-		)
-		(stroke
-			(width 0)
-			(type default)
-		)
-	)
-	(wire
-		(pts
 			(xy 232.41 78.74) (xy 232.41 69.85)
 		)
@@
 	(wire
 		(pts
+			(xy 115.57 153.67) (xy 106.68 153.67)
+		)
+		(stroke
+			(width 0)
+			(type default)
+		)
+	)
+	(wire
+		(pts
 			(xy 118.11 62.23) (xy 129.54 62.23)
 		)
@@
 	(wire
 		(pts
-			(xy 115.57 153.67) (xy 106.68 153.67)
-		)
-		(stroke
-			(width 0)
-			(type default)
-		)
-	)
-	(wire
-		(pts
 			(xy 102.87 90.17) (xy 104.14 90.17)
 		)
@@
 		(pts
 			(xy 215.9 148.59) (xy 224.79 148.59)
-		)
-		(stroke
-			(width 0)
-			(type default)
-		)
-	)
-	(wire
-		(pts
-			(xy 106.68 153.67) (xy 106.68 156.21)
 		)
 		(stroke
@@
 			)
 		)
-		(property "Footprint" "Hyper_Wheel:SW_KS33_HS_KS-2P02B01-02_HS_1u"
+		(property "Footprint" "Hyper_Wheel:SW_KS33_1u"
 			(at 259.08 81.28 0)
 			(hide yes)
@@
 	)
 	(symbol
+		(lib_id "Connector:Conn_01x04_Socket")
+		(at 101.6 161.29 180)
+		(unit 1)
+		(body_style 1)
+		(exclude_from_sim no)
+		(in_bom yes)
+		(on_board yes)
+		(in_pos_files yes)
+		(dnp no)
+		(property "Reference" "J2-1"
+			(at 105.41 148.844 0)
+			(show_name no)
+			(do_not_autoplace no)
+			(effects
+				(font
+					(size 1.27 1.27)
+				)
+				(justify left)
+			)
+		)
+		(property "Value" "Conn_01x04_Socket"
+			(at 101.346 147.574 0)
+			(show_name no)
+			(do_not_autoplace no)
+			(effects
+				(font
+					(size 1.27 1.27)
+				)
+				(justify left)
+			)
+		)
+		(property "Footprint" "Connector_JST:JST_EH_S4B-EH_1x04_P2.50mm_Horizontal"
+			(at 101.6 161.29 0)
+			(hide yes)
+			(show_name no)
+			(do_not_autoplace no)
+			(effects
+				(font
+					(size 1.27 1.27)
+				)
+			)
+		)
+		(property "Datasheet" ""
+			(at 101.6 161.29 0)
+			(hide yes)
+			(show_name no)
+			(do_not_autoplace no)
+			(effects
+				(font
+					(size 1.27 1.27)
+				)
+			)
+		)
+		(property "Description" "Generic connector, single row, 01x04, script generated"
+			(at 101.6 161.29 0)
+			(hide yes)
+			(show_name no)
+			(do_not_autoplace no)
+			(effects
+				(font
+					(size 1.27 1.27)
+				)
+			)
+		)
+		(property "KiLib_Generator" "connector/pin_header_socket"
+			(at 101.6 161.29 0)
+			(hide yes)
+			(show_name no)
+			(do_not_autoplace no)
+			(effects
+				(font
+					(size 1.27 1.27)
+				)
+			)
+		)
+		(pin "3"
+		)
+		(pin "4"
+		)
+		(pin "1"
+		)
+		(pin "2"
+		)
+		(instances
+			(project "Hyper_Wheel_XIAO"
+				(path "/3f05eeb1-03f9-49d1-8a58-0bc3d5427d25/27e14a4a-7907-4947-a1bd-66ab05fca5b6"
+					(reference "J2-1")
+					(unit 1)
+				)
+			)
+		)
+	)
+	(symbol
 		(lib_id "power:GND")
 		(at 163.83 58.42 0)
@@
 	)
 	(symbol
-		(lib_id "Connector:Conn_01x04_Socket")
-		(at 101.6 161.29 180)
-		(unit 1)
-		(body_style 1)
-		(exclude_from_sim no)
-		(in_bom yes)
-		(on_board yes)
-		(in_pos_files yes)
-		(dnp no)
-		(property "Reference" "J2-1"
-			(at 101.346 150.114 0)
-			(show_name no)
-			(do_not_autoplace no)
-			(effects
-				(font
-					(size 1.27 1.27)
-				)
-				(justify left)
-			)
-		)
-		(property "Value" "Conn_01x04_Socket"
-			(at 101.346 147.574 0)
-			(show_name no)
-			(do_not_autoplace no)
-			(effects
-				(font
-					(size 1.27 1.27)
-				)
-				(justify left)
-			)
-		)
-		(property "Footprint" "Connector_PinHeader_2.54mm:PinHeader_1x04_P2.54mm_Vertical"
-			(at 101.6 161.29 0)
-			(hide yes)
-			(show_name no)
-			(do_not_autoplace no)
-			(effects
-				(font
-					(size 1.27 1.27)
-				)
-			)
-		)
-		(property "Datasheet" ""
-			(at 101.6 161.29 0)
-			(hide yes)
-			(show_name no)
-			(do_not_autoplace no)
-			(effects
-				(font
-					(size 1.27 1.27)
-				)
-			)
-		)
-		(property "Description" "Generic connector, single row, 01x04, script generated"
-			(at 101.6 161.29 0)
-			(hide yes)
-			(show_name no)
-			(do_not_autoplace no)
-			(effects
-				(font
-					(size 1.27 1.27)
-				)
-			)
-		)
-		(property "KiLib_Generator" "connector/pin_header_socket"
-			(at 101.6 161.29 0)
-			(hide yes)
-			(show_name no)
-			(do_not_autoplace no)
-			(effects
-				(font
-					(size 1.27 1.27)
-				)
-			)
-		)
-		(pin "3"
-		)
-		(pin "4"
-		)
-		(pin "1"
-		)
-		(pin "2"
-		)
-		(instances
-			(project "Hyper_Wheel_XIAO"
-				(path "/3f05eeb1-03f9-49d1-8a58-0bc3d5427d25/27e14a4a-7907-4947-a1bd-66ab05fca5b6"
-					(reference "J2-1")
-					(unit 1)
-				)
-			)
-		)
-	)
-	(symbol
 		(lib_id "Connector:Conn_01x06_Pin")
 		(at 134.62 62.23 0)
@@
 			)
 		)
-		(property "Footprint" "Hyper_Wheel:SW_KS33_HS_KS-2P02B01-02_HS_1u"
+		(property "Footprint" "Hyper_Wheel:SW_KS33_1u"
 			(at 234.95 57.15 0)
 			(hide yes)
@@
 			)
 		)
-		(property "Footprint" "Hyper_Wheel:SW_KS33_HS_KS-2P02B01-02_HS_1u"
+		(property "Footprint" "Hyper_Wheel:SW_KS33_1u"
 			(at 246.38 57.15 0)
 			(hide yes)
@@
 			)
 		)
-		(property "Footprint" "Hyper_Wheel:SW_KS33_HS_KS-2P02B01-02_HS_1u"
+		(property "Footprint" "Hyper_Wheel:SW_KS33_1u"
 			(at 247.65 81.28 0)
 			(hide yes)
@@
 			)
 		)
-		(property "Footprint" "Hyper_Wheel:SW_KS33_HS_KS-2P02B01-02_HS_1u"
+		(property "Footprint" "Hyper_Wheel:SW_KS33_1u"
 			(at 220.98 57.15 0)
 			(hide yes)
@@
 			)
 		)
-		(property "Footprint" "Hyper_Wheel:SW_KS33_HS_KS-2P02B01-02_HS_1u"
+		(property "Footprint" "Hyper_Wheel:SW_KS33_1u"
 			(at 222.25 81.28 0)
 			(hide yes)
@@
 			)
 		)
-		(property "Footprint" "Hyper_Wheel:SW_KS33_HS_KS-2P02B01-02_HS_1u"
+		(property "Footprint" "Hyper_Wheel:SW_KS33_1u"
 			(at 234.95 81.28 0)
 			(hide yes)
@@
 			)
 		)
-		(property "Footprint" "Connector_PinHeader_2.54mm:PinHeader_1x06_P2.54mm_Vertical"
+		(property "Footprint" "Connector_JST:JST_EH_S6B-EH_1x06_P2.50mm_Horizontal"
 			(at 138.43 62.23 0)
 			(hide yes)
@@
 			)
 		)
-		(property "Footprint" "Hyper_Wheel:SW_KS33_HS_KS-2P02B01-02_HS_1u"
+		(property "Footprint" "Hyper_Wheel:SW_KS33_1u"
 			(at 257.81 57.15 0)
 			(hide yes)
