File: PCB/Hyper_Wheel_XIAO/PowerBoard.kicad_sch (KiCad schematic)
At the start: 12 parts, among them J2 LIPO, U1 CSD85301Q2, U6 BQ29700DSER, U9 CSD85301Q2

Commit message: RevB Xiao Updates. Fab
Parts:
- J2: footprint Connector_JST:JST_EH_B2B-EH-A_1x02_P2.50mm_Vertical -> Connector_JST:JST_EH_S2B-EH_1x02_P2.50mm_Horizontal
Changed lines of the file:
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@@
 			)
 		)
-		(property "Footprint" "Connector_JST:JST_EH_B2B-EH-A_1x02_P2.50mm_Vertical"
+		(property "Footprint" "Connector_JST:JST_EH_S2B-EH_1x02_P2.50mm_Horizontal"
 			(at 265.43 87.63 0)
 			(hide yes)
